Commit message: Change the lidar sensor so that ray 0 elevation, 0 azimuth is the z axis instead of the x
This matches hardware

File: mujoco_ros2_control_demos/demo_resources/robot/3d_lidar_robot.urdf (robot description, URDF)
Before this commit: robot two_dof_robot, 13 links, 12 joints
Links:
- removed link lidar_sensor_frame
- added link front_lidar
- added link front_lidar_sensor_frame
Joints:
- removed joint lidar_sensor_link
- added joint front_lidar_link: type fixed, parent world, child front_lidar, origin xyz=1.0 2.0 0 rpy=0 0 -1.5708
- added joint front_lidar_sensor_frame: type fixed, parent front_lidar, child front_lidar_sensor_frame, origin xyz=0.0 0.0 0.15 rpy=0 -1.5708 -1.5708

Commit message: I was wrong about the normal direction of the rays.  Should be x

File: mujoco_ros2_control_demos/demo_resources/robot/3d_lidar_robot.urdf (robot description, URDF)
Before this commit: robot two_dof_robot, 14 links, 13 joints
Links:
- removed link front_lidar
- removed link front_lidar_sensor_frame
- added link front_lidar_frame
Joints:
- removed joint front_lidar_sensor_frame
- joint front_lidar_link: child front_lidar -> front_lidar_frame; origin xyz=1.0 2.0 0 rpy=0 0 -1.5708 -> xyz=1.0 2.0 0.0 rpy=0 0 -1.5708
